Commit message: added encoders

File: trilosaurus_description/urdf/trilosaurus_description.urdf.xacro (robot description, xacro)
@@ -4,11 +4,11 @@
   <!-- Constants for robot dimensions -->
   <xacro:property name="PI" value="3.1415926535897931"/>
-  <xacro:property name="base_mass" value="0.3" /> <!-- arbitrary value for base mass -->
+  <xacro:property name="base_mass" value="0.1" /> <!-- arbitrary value for base mass -->
   <xacro:property name="base_width" value="0.1" />
   <xacro:property name="base_length" value="0.1" />
   <xacro:property name="base_height" value="0.05" />
-  <xacro:property name="wheel_mass" value="0.3" /> <!-- arbitrary value for wheel mass -->
+  <xacro:property name="wheel_mass" value="0.1" /> <!-- arbitrary value for wheel mass -->
   <xacro:property name="wheel_len" value="0.020" />
-  <xacro:property name="wheel_radius" value="0.015" />
+  <xacro:property name="wheel_radius" value="0.021" />
   <xacro:property name="caster_wheel_mass" value="0.1" /> <!-- arbitrary value for caster wheel mass -->
   <xacro:property name="caster_wheel_radius" value="0.015" />
@@ -38,8 +38,24 @@
       </inertial>
     </link>
+    <!-- marker -->
+    <link name="_marker">
+      <visual>
+	<origin xyz="0.06 0 0.05" rpy="0 0 0"/>
+	<geometry>
+          <box size="0.02 0.01 0.005"/>
+	</geometry>
+	<material name="white"/>
+      </visual>
+    </link>
+    <joint name="marker_joint" type="fixed">
+      <parent link="${prefix}base_link"/>
+      <child link="_marker"/>
+      <origin xyz="0 0 0" rpy="0 0 0"/>
+    </joint>
+    <!-- left wheel -->
     <joint name="${prefix}left_wheel_joint" type="continuous">
       <parent link="${prefix}base_link"/>
       <child link="${prefix}left_wheel"/>
-      <origin xyz="0 -${base_width/2} ${z_offset}" rpy="0 0 0"/>
+      <origin xyz="0 ${base_width/2} ${z_offset}" rpy="0 0 0"/>
       <axis xyz="0 1 0"/>
       <dynamics damping="0.2"/>
@@ -69,8 +85,9 @@
         </inertial>
       </link>
+    <!-- right wheel -->
     <joint name="${prefix}right_wheel_joint" type="continuous">
       <parent link="${prefix}base_link"/>
       <child link="${prefix}right_wheel"/>
-      <origin xyz="0 ${base_width/2} ${z_offset}" rpy="0 0 0"/>
+      <origin xyz="0 -${base_width/2} ${z_offset}" rpy="0 0 0"/>
       <axis xyz="0 1 0"/>
       <dynamics damping="0.2"/>

Commit message: lidar and vision starting to work in ros2

File: trilosaurus_description/urdf/trilosaurus_description.urdf.xacro (robot description, xacro)
@@ -38,4 +38,12 @@
       </inertial>
     </link>
+    <!-- Footprint -->
+    <link name="${prefix}base_footprint">
+    </link>
+    <joint name="base_footprint_joint" type="fixed">
+      <parent link="${prefix}base_link"/>
+      <child link="${prefix}base_footprint"/>
+      <origin xyz="0 0 -${base_height}" rpy="0 0 0"/>
+  </joint>
     <!-- marker -->
     <link name="_marker">
@@ -53,4 +61,34 @@
       <origin xyz="0 0 0" rpy="0 0 0"/>
     </joint>
+    <!-- IMU -->
+    <link name="imu_link">
+      <visual>
+	<origin xyz="0 0 0.05" rpy="0 0 0"/>
+	<geometry>
+          <box size="0.005 0.005 0.005"/>
+	</geometry>
+	<material name="white"/>
+      </visual>
+    </link>
+    <joint name="imu_joint" type="fixed">
+      <parent link="${prefix}base_link"/>
+      <child link="imu_link"/>
+      <origin xyz="0 0 0" rpy="0 0 0"/>
+    </joint>
+   <!-- LIDAR -->
+    <link name="laser_link">
+      <visual>
+	<origin xyz="0 0 0.1" rpy="0 0 0"/>
+	<geometry>
+          <box size="0.005 0.005 0.005"/>
+	</geometry>
+	<material name="white"/>
+      </visual>
+    </link>
+    <joint name="laser_joint" type="fixed">
+      <parent link="${prefix}base_link"/>
+      <child link="laser_link"/>
+      <origin xyz="0 0 0" rpy="0 0 ${PI}"/>
+    </joint>
     <!-- left wheel -->
     <joint name="${prefix}left_wheel_joint" type="continuous">
